Commit message: Removed official Petoi mdoel and replaced with simplified model. Lots of other changes

File: bittle_description/urdf/bittle.xacro (robot description, xacro)
@@ -1,2297 +1,326 @@
-<?xml version="1.0" ?>
-<robot name="bittle" xmlns:xacro="http://www.ros.org/wiki/xacro">
-<xacro:include filename="$(find bittle_description)/urdf/materials.xacro" />
-<xacro:include filename="$(find bittle_description)/urdf/bittle.trans" />
-<xacro:include filename="$(find bittle_description)/urdf/bittle.gazebo" />
-<link name="base_link">
-  <inertial>
-    <origin xyz="0.002168345924058267 4.1430032450566535e-08 0.02555254458454454" rpy="0 0 0"/>
-    <mass value="0.01989030949409733"/>
-    <inertia ixx="1.5e-05" iyy="2.4e-05" izz="3.8e-05" ixy="0.0" iyz="0.0" ixz="-0.0"/>
-  </inertial>
-  <visual>
-    <origin xyz="0 0 0" rpy="0 0 0"/>
-    <geometry>
-      <mesh filename="package://bittle_description/meshes/base_link.stl" scale="0.001 0.001 0.001"/>
-    </geometry>
-    <material name="silver"/>
-  </visual>
-  <collision>
-    <origin xyz="0 0 0" rpy="0 0 0"/>
-    <geometry>
-      <mesh filename="package://bittle_description/meshes/base_link.stl" scale="0.001 0.001 0.001"/>
-    </geometry>
-  </collision>
-</link>
-<link name="front__1">
-  <inertial>
-    <origin xyz="-0.00995696017036956 0.02800119957987551 -0.0005395302490400072" rpy="0 0 0"/>
-    <mass value="0.0039123866206911126"/>
-    <inertia ixx="2e-06" iyy="1e-06" izz="2e-06" ixy="0.0" iyz="-0.0" ixz="0.0"/>
-  </inertial>
-  <visual>
-    <origin xyz="-0.061733 0.028 -0.025792" rpy="0 0 0"/>
-    <geometry>
-      <mesh filename="package://bittle_description/meshes/front__1.stl" scale="0.001 0.001 0.001"/>
-    </geometry>
-    <material name="silver"/>
-  </visual>
-  <collision>
-    <origin xyz="-0.061733 0.028 -0.025792" rpy="0 0 0"/>
-    <geometry>
-      <mesh filename="package://bittle_description/meshes/front__1.stl" scale="0.001 0.001 0.001"/>
-    </geometry>
-  </collision>
-</link>
-<link name="rear__1">
-  <inertial>
-    <origin xyz="0.009956960170745259 -0.027998805995973614 -0.0005395302462037725" rpy="0 0 0"/>
-    <mass value="0.003912386618757239"/>
-    <inertia ixx="2e-06" iyy="1e-06" izz="2e-06" ixy="-0.0" iyz="-0.0" ixz="-0.0"/>
-  </inertial>
-  <visual>
-    <origin xyz="0.061733 -0.028 -0.025792" rpy="0 0 0"/>
-    <geometry>
-      <mesh filename="package://bittle_description/meshes/rear__1.stl" scale="0.001 0.001 0.001"/>
-    </geometry>
-    <material name="silver"/>
-  </visual>
-  <collision>
-    <origin xyz="0.061733 -0.028 -0.025792" rpy="0 0 0"/>
-    <geometry>
-      <mesh filename="package://bittle_description/meshes/rear__1.stl" scale="0.001 0.001 0.001"/>
-    </geometry>
-  </collision>
-</link>
-<link name="servo_rfs_1">
-  <inertial>
-    <origin xyz="-0.012134511463850035 0.0033276213458265785 0.007005695786782645" rpy="0 0 0"/>
-    <mass value="0.016198785326804743"/>
-    <inertia ixx="1e-06" iyy="1e-06" izz="1e-06" ixy="0.0" iyz="-0.0" ixz="0.0"/>
-  </inertial>
-  <visual>
-    <origin xyz="-0.059645 0.036 -0.017875" rpy="0 0 0"/>
-    <geometry>
-      <mesh filename="package://bittle_description/meshes/servo_rfs_1.stl" scale="0.001 0.001 0.001"/>
-    </geometry>
-    <material name="silver"/>
-  </visual>
-  <collision>
-    <origin xyz="-0.059645 0.036 -0.017875" rpy="0 0 0"/>
-    <geometry>
-      <mesh filename="package://bittle_description/meshes/servo_rfs_1.stl" scale="0.001 0.001 0.001"/>
-    </geometry>
-  </collision>
-</link>
-<link name="servo_rrs__1">
-  <inertial>
-    <origin xyz="0.012134511463850035 0.0033276213458265508 0.007005695786782652" rpy="0 0 0"/>
-    <mass value="0.016198785326804747"/>
-    <inertia ixx="1e-06" iyy="1e-06" izz="1e-06" ixy="-0.0" iyz="-0.0" ixz="-0.0"/>
-  </inertial>
-  <visual>
-    <origin xyz="0.059645 0.036 -0.017875" rpy="0 0 0"/>
-    <geometry>
-      <mesh filename="package://bittle_description/meshes/servo_rrs__1.stl" scale="0.001 0.001 0.001"/>
-    </geometry>
-    <material name="silver"/>
-  </visual>
-  <collision>
-    <origin xyz="0.059645 0.036 -0.017875" rpy="0 0 0"/>
-    <geometry>
-      <mesh filename="package://bittle_description/meshes/servo_rrs__1.stl" scale="0.001 0.001 0.001"/>
-    </geometry>
-  </collision>
-</link>
-<link name="c_neck__1">
-  <inertial>
-    <origin xyz="0.0003476160573467474 8.689791074277334e-16 0.0015392691836189978" rpy="0 0 0"/>
-    <mass value="0.0002786420162302464"/>
-    <inertia ixx="0.0" iyy="0.0" izz="0.0" ixy="0.0" iyz="-0.0" ixz="0.0"/>
-  </inertial>
-  <visual>
-    <origin xyz="-0.044904 -0.0 -0.031351" rpy="0 0 0"/>
-    <geometry>
-      <mesh filename="package://bittle_description/meshes/c_neck__1.stl" scale="0.001 0.001 0.001"/>
-    </geometry>
-    <material name="silver"/>
-  </visual>
-  <collision>
-    <origin xyz="-0.044904 -0.0 -0.031351" rpy="0 0 0"/>
-    <geometry>
-      <mesh filename="package://bittle_description/meshes/c_neck__1.stl" scale="0.001 0.001 0.001"/>
-    </geometry>
-  </collision>
-</link>
-<link name="head__1">
-  <inertial>
-    <origin xyz="0.01773367569221658 0.010875428717563109 0.005303020015208416" rpy="0 0 0"/>
-    <mass value="0.0047175875144439645"/>
-    <inertia ixx="1e-06" iyy="1e-06" izz="1e-06" ixy="0.0" iyz="-0.0" ixz="0.0"/>
-  </inertial>
-  <visual>
-    <origin xyz="-0.055711 0.017155 -0.060327" rpy="0 0 0"/>
-    <geometry>
-      <mesh filename="package://bittle_description/meshes/head__1.stl" scale="0.001 0.001 0.001"/>
-    </geometry>
-    <material name="silver"/>
-  </visual>
-  <collision>
-    <origin xyz="-0.055711 0.017155 -0.060327" rpy="0 0 0"/>
-    <geometry>
-      <mesh filename="package://bittle_description/meshes/head__1.stl" scale="0.001 0.001 0.001"/>
-    </geometry>
-  </collision>
-</link>
-<link name="jaw_1">
-  <inertial>
-    <origin xyz="-0.0009535400770716435 0.0073141018408541866 0.015990572203006634" rpy="0 0 0"/>
-    <mass value="0.00390701419929372"/>
-    <inertia ixx="1e-06" iyy="1e-06" izz="1e-06" ixy="0.0" iyz="0.0" ixz="0.0"/>
-  </inertial>
-  <visual>
-    <origin xyz="-0.06445 0.012925 -0.034027" rpy="0 0 0"/>
-    <geometry>
-      <mesh filename="package://bittle_description/meshes/jaw_1.stl" scale="0.001 0.001 0.001"/>
-    </geometry>
-    <material name="silver"/>
-  </visual>
-  <collision>
-    <origin xyz="-0.06445 0.012925 -0.034027" rpy="0 0 0"/>
-    <geometry>
-      <mesh filename="package://bittle_description/meshes/jaw_1.stl" scale="0.001 0.001 0.001"/>
-    </geometry>
-  </collision>
-</link>
-<link name="tho_rf__1">
-  <inertial>
-    <origin xyz="-0.020399619281867152 -1.772774812243416e-05 -0.0054647510340394435" rpy="0 0 0"/>
-    <mass value="0.0016124935043948178"/>
-    <inertia ixx="0.0" iyy="0.0" izz="0.0" ixy="-0.0" iyz="-0.0" ixz="-0.0"/>
-  </inertial>
-  <visual>
-    <origin xyz="-0.038977 0.050355 -0.018377" rpy="0 0 0"/>
-    <geometry>
-      <mesh filename="package://bittle_description/meshes/tho_rf__1.stl" scale="0.001 0.001 0.001"/>
-    </geometry>
-    <material name="silver"/>
-  </visual>
-  <collision>
-    <origin xyz="-0.038977 0.050355 -0.018377" rpy="0 0 0"/>
-    <geometry>
-      <mesh filename="package://bittle_description/meshes/tho_rf__1.stl" scale="0.001 0.001 0.001"/>
-    </geometry>
-  </collision>
-</link>
-<link name="servo_neck__1">
-  <inertial>
-    <origin xyz="0.01000501101063378 -0.0036770959380430985 0.008458014805728817" rpy="0 0 0"/>
-    <mass value="0.016198785326804754"/>
-    <inertia ixx="1e-06" iyy="1e-06" izz="1e-06" ixy="0.0" iyz="-0.0" ixz="-0.0"/>
-  </inertial>
-  <visual>
-    <origin xyz="-0.047554 -0.0 -0.035941" rpy="0 0 0"/>
-    <geometry>
-      <mesh filename="package://bittle_description/meshes/servo_neck__1.stl" scale="0.001 0.001 0.001"/>
-    </geometry>
-    <material name="silver"/>
-  </visual>
-  <collision>
-    <origin xyz="-0.047554 -0.0 -0.035941" rpy="0 0 0"/>
-    <geometry>
-      <mesh filename="package://bittle_description/meshes/servo_neck__1.stl" scale="0.001 0.001 0.001"/>
-    </geometry>
-  </collision>
-</link>
-<link name="tube__1">
-  <inertial>
-    <origin xyz="0.0011153307229088694 0.005350015413290346 -0.004241660835567474" rpy="0 0 0"/>
-    <mass value="0.0008476319886892588"/>
-    <inertia ixx="0.0" iyy="0.0" izz="0.0" ixy="-0.0" iyz="-0.0" ixz="-0.0"/>
-  </inertial>
-  <visual>
-    <origin xyz="-0.02915 0.052607 -0.02028" rpy="0 0 0"/>
-    <geometry>
-      <mesh filename="package://bittle_description/meshes/tube__1.stl" scale="0.001 0.001 0.001"/>
-    </geometry>
-    <material name="silver"/>
-  </visual>
-  <collision>
-    <origin xyz="-0.02915 0.052607 -0.02028" rpy="0 0 0"/>
-    <geometry>
-      <mesh filename="package://bittle_description/meshes/tube__1.stl" scale="0.001 0.001 0.001"/>
-    </geometry>
-  </collision>
-</link>
-<link name="th_rf_1">
-  <inertial>
-    <origin xyz="-0.01050527468812052 0.0005245346031438683 -0.0028130983482547826" rpy="0 0 0"/>
-    <mass value="0.0016124994656611404"/>
-    <inertia ixx="0.0" iyy="0.0" izz="0.0" ixy="-0.0" iyz="-0.0" ixz="-0.0"/>
-  </inertial>
-  <visual>
-    <origin xyz="-0.0525 0.0508 -0.022" rpy="0 0 0"/>
-    <geometry>
-      <mesh filename="package://bittle_description/meshes/th_rf_1.stl" scale="0.001 0.001 0.001"/>
-    </geometry>
-    <material name="silver"/>
-  </visual>
-  <collision>
-    <origin xyz="-0.0525 0.0508 -0.022" rpy="0 0 0"/>
-    <geometry>
-      <mesh filename="package://bittle_description/meshes/th_rf_1.stl" scale="0.001 0.001 0.001"/>
-    </geometry>
-  </collision>
-</link>
-<link name="c_thorf_1">
-  <inertial>
-    <origin xyz="0.0004222776002216107 0.003991736806568551 0.00011331940655908042" rpy="0 0 0"/>
-    <mass value="0.0003202445573374636"/>
-    <inertia ixx="0.0" iyy="0.0" izz="0.0" ixy="0.0" iyz="0.0" ixz="-0.0"/>
-  </inertial>
-  <visual>
-    <origin xyz="-0.008067 0.054937 -0.010094" rpy="0 0 0"/>
-    <geometry>
-      <mesh filename="package://bittle_description/meshes/c_thorf_1.stl" scale="0.001 0.001 0.001"/>
-    </geometry>
-    <material name="silver"/>
-  </visual>
-  <collision>
-    <origin xyz="-0.008067 0.054937 -0.010094" rpy="0 0 0"/>
-    <geometry>
-      <mesh filename="package://bittle_description/meshes/c_thorf_1.stl" scale="0.001 0.001 0.001"/>
-    </geometry>
-  </collision>
-</link>
-<link name="servo_lfs_1">
-  <inertial>
-    <origin xyz="-0.012134511463850035 -0.0033276213458265855 0.007005695786782638" rpy="0 0 0"/>
-    <mass value="0.016198785326804747"/>
-    <inertia ixx="1e-06" iyy="1e-06" izz="1e-06" ixy="-0.0" iyz="0.0" ixz="0.0"/>
-  </inertial>
-  <visual>
-    <origin xyz="-0.059645 -0.036 -0.017875" rpy="0 0 0"/>
-    <geometry>
-      <mesh filename="package://bittle_description/meshes/servo_lfs_1.stl" scale="0.001 0.001 0.001"/>
-    </geometry>
-    <material name="silver"/>
-  </visual>
-  <collision>
-    <origin xyz="-0.059645 -0.036 -0.017875" rpy="0 0 0"/>
-    <geometry>
-      <mesh filename="package://bittle_description/meshes/servo_lfs_1.stl" scale="0.001 0.001 0.001"/>
-    </geometry>
-  </collision>
-</link>
-<link name="servo_lrs__1">
-  <inertial>
-    <origin xyz="0.012134511463850021 -0.0033276213458265577 0.007005695786782652" rpy="0 0 0"/>
-    <mass value="0.006359523128301122"/>
-    <inertia ixx="0.0" iyy="0.0" izz="0.0" ixy="0.0" iyz="0.0" ixz="-0.0"/>
-  </inertial>
-  <visual>
-    <origin xyz="0.059645 -0.036 -0.017875" rpy="0 0 0"/>
-    <geometry>
-      <mesh filename="package://bittle_description/meshes/servo_lrs__1.stl" scale="0.001 0.001 0.001"/>
-    </geometry>
-    <material name="silver"/>
-  </visual>
-  <collision>
-    <origin xyz="0.059645 -0.036 -0.017875" rpy="0 0 0"/>
-    <geometry>
-      <mesh filename="package://bittle_description/meshes/servo_lrs__1.stl" scale="0.001 0.001 0.001"/>
-    </geometry>
-  </collision>
-</link>
-<link name="a_1">
-  <inertial>
-    <origin xyz="0.0011980267759206685 0.00010035438122205087 -0.0010926527391464588" rpy="0 0 0"/>
-    <mass value="9.845210937902234e-06"/>
-    <inertia ixx="0.0" iyy="0.0" izz="0.0" ixy="0.0" iyz="-0.0" ixz="-0.0"/>
-  </inertial>
-  <visual>
-    <origin xyz="0.006412 0.032855 -0.027034" rpy="0 0 0"/>
-    <geometry>
-      <mesh filename="package://bittle_description/meshes/a_1.stl" scale="0.001 0.001 0.001"/>
-    </geometry>
-    <material name="silver"/>
-  </visual>
-  <collision>
-    <origin xyz="0.006412 0.032855 -0.027034" rpy="0 0 0"/>
-    <geometry>
-      <mesh filename="package://bittle_description/meshes/a_1.stl" scale="0.001 0.001 0.001"/>
-    </geometry>
-  </collision>
-</link>
-<link name="b__1">
-  <inertial>
-    <origin xyz="0.0012604376192366716 9.955965670559869e-05 -0.0005822422676032835" rpy="0 0 0"/>
-    <mass value="7.636356391604399e-06"/>
-    <inertia ixx="0.0" iyy="0.0" izz="0.0" ixy="-0.0" iyz="-0.0" ixz="-0.0"/>
-  </inertial>
-  <visual>
-    <origin xyz="0.002835 0.03277 -0.025616" rpy="0 0 0"/>
-    <geometry>
-      <mesh filename="package://bittle_description/meshes/b__1.stl" scale="0.001 0.001 0.001"/>
-    </geometry>
-    <material name="silver"/>
-  </visual>
-  <collision>
-    <origin xyz="0.002835 0.03277 -0.025616" rpy="0 0 0"/>
-    <geometry>
-      <mesh filename="package://bittle_description/meshes/b__1.stl" scale="0.001 0.001 0.001"/>
-    </geometry>
-  </collision>
-</link>
-<link name="c_1">
-  <inertial>
-    <origin xyz="0.0004800725906685088 0.00010010236221810742 -0.0014636091148647126" rpy="0 0 0"/>
-    <mass value="5.729215470952315e-06"/>
-    <inertia ixx="0.0" iyy="0.0" izz="0.0" ixy="0.0" iyz="-0.0" ixz="0.0"/>
-  </inertial>
-  <visual>
-    <origin xyz="-0.000594 0.032751 -0.026875" rpy="0 0 0"/>
-    <geometry>
-      <mesh filename="package://bittle_description/meshes/c_1.stl" scale="0.001 0.001 0.001"/>
-    </geometry>
-    <material name="silver"/>
-  </visual>
-  <collision>
-    <origin xyz="-0.000594 0.032751 -0.026875" rpy="0 0 0"/>
-    <geometry>
-      <mesh filename="package://bittle_description/meshes/c_1.stl" scale="0.001 0.001 0.001"/>
-    </geometry>
-  </collision>
-</link>
-<link name="d_1">
-  <inertial>
-    <origin xyz="0.0013568994912427604 9.998382103230258e-05 -0.0006094898025702025" rpy="0 0 0"/>
-    <mass value="7.529988845478445e-06"/>
-    <inertia ixx="0.0" iyy="0.0" izz="0.0" ixy="0.0" iyz="-0.0" ixz="0.0"/>
-  </inertial>
-  <visual>
-    <origin xyz="-0.002348 0.032764 -0.025618" rpy="0 0 0"/>
-    <geometry>
-      <mesh filename="package://bittle_description/meshes/d_1.stl" scale="0.001 0.001 0.001"/>
-    </geometry>
-    <material name="silver"/>
-  </visual>
-  <collision>
-    <origin xyz="-0.002348 0.032764 -0.025618" rpy="0 0 0"/>
-    <geometry>
-      <mesh filename="package://bittle_description/meshes/d_1.stl" scale="0.001 0.001 0.001"/>
-    </geometry>
-  </collision>
-</link>
-<link name="e_1">
-  <inertial>
-    <origin xyz="0.00036682874729430416 0.00010009700467959737 -0.0010508795807335665" rpy="0 0 0"/>
-    <mass value="3.2406127639379744e-06"/>
-    <inertia ixx="0.0" iyy="0.0" izz="0.0" ixy="-0.0" iyz="-0.0" ixz="0.0"/>
-  </inertial>
-  <visual>
-    <origin xyz="-0.005742 0.032834 -0.026061" rpy="0 0 0"/>
-    <geometry>
-      <mesh filename="package://bittle_description/meshes/e_1.stl" scale="0.001 0.001 0.001"/>
-    </geometry>
-    <material name="silver"/>
-  </visual>
-  <collision>
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